Commit message: Tweaks for Elsabot 4wd base

File: linorobot2_description/urdf/4wd_properties.urdf.xacro (robot description, xacro)
@@ -1,17 +1,17 @@
 <?xml version="1.0"?>
 <robot xmlns:xacro="http://ros.org/wiki/xacro">
-  <xacro:property name="base_length" value="0.445" />
-  <xacro:property name="base_width" value="0.200" />
-  <xacro:property name="base_height" value="0.129" />
+  <xacro:property name="base_length" value="0.510" />
+  <xacro:property name="base_width" value="0.318" />
+  <xacro:property name="base_height" value="0.180" />
   <xacro:property name="base_mass" value="10" />
-  <xacro:property name="wheel_radius" value="0.07162" />
-  <xacro:property name="wheel_width" value="0.05" />
-  <xacro:property name="wheel_pos_x" value="0.120" />
-  <xacro:property name="wheel_pos_y" value="0.1355" />
-  <xacro:property name="wheel_pos_z" value="-0.04788" />
+  <xacro:property name="wheel_radius" value="0.078" />
+  <xacro:property name="wheel_width" value="0.047" />
+  <xacro:property name="wheel_pos_x" value="0.1505" />
+  <xacro:property name="wheel_pos_y" value="0.1925" />
+  <xacro:property name="wheel_pos_z" value="-0.012" />
   <xacro:property name="wheel_mass" value=".6" />
-  <xacro:property name="wheel_torque" value="20" />
+  <xacro:property name="wheel_torque" value="12" />
   <xacro:property name="laser_pose">
-    <origin xyz="-0.0475 0 0.125" rpy="0 0 0"/>
+    <origin xyz="0.205 0 0.156" rpy="0 0 3.14"/>
   </xacro:property>
   <xacro:property name="depth_sensor_pose">

Commit message: Fine tune positions, add oakd camera, and add meshes for base and oakd

File: linorobot2_description/urdf/4wd_properties.urdf.xacro (robot description, xacro)
@@ -5,13 +5,13 @@
   <xacro:property name="base_height" value="0.180" />
   <xacro:property name="base_mass" value="10" />
-  <xacro:property name="wheel_radius" value="0.078" />
+  <xacro:property name="wheel_radius" value="0.0795" />
   <xacro:property name="wheel_width" value="0.047" />
   <xacro:property name="wheel_pos_x" value="0.1505" />
   <xacro:property name="wheel_pos_y" value="0.1925" />
-  <xacro:property name="wheel_pos_z" value="-0.012" />
+  <xacro:property name="wheel_pos_z" value="-0.1105" />
   <xacro:property name="wheel_mass" value=".6" />
   <xacro:property name="wheel_torque" value="12" />
   <xacro:property name="laser_pose">
-    <origin xyz="0.205 0 0.156" rpy="0 0 3.14"/>
+    <origin xyz="0.205 0 0.064" rpy="0 0 3.14"/>
   </xacro:property>
   <xacro:property name="depth_sensor_pose">

File: linorobot2_description/urdf/mech/base.urdf.xacro (robot description, xacro)
@@ -7,9 +7,9 @@
         <origin xyz="0 0 0" rpy="0 0 0"/>
         <geometry>
-          <box size="${length} ${width} ${height}"/>
-          <!-- <mesh filename="" scale="0.001 0.001 0.001"/> -->
+          <!-- box size="${length} ${width} ${height}"/ -->
+          <mesh filename="package://linorobot2_description/meshes/elsabot_4wd.stl" scale="1.0 1.0 1.0"/> -->
         </geometry>
-        <material name="yellow">
-          <color rgba="0.8784 0.6627 0.6627 1.0"/>
+        <material name="gray">
+          <color rgba="0.8 0.8 0.8 1.0"/>
         </material>
       </visual>

File: linorobot2_description/urdf/mech/wheel.urdf.xacro (robot description, xacro)
@@ -6,5 +6,5 @@
         <origin xyz="0 0 0" rpy="${pi/2} 0 0"/>
         <geometry>
-          <cylinder radius="${radius}" length="${width}"/>
+          <!--cylinder radius="${radius}" length="${width}"/-->
         </geometry>
         <material name="blue">

File: linorobot2_description/urdf/robots/4wd.urdf.xacro (robot description, xacro)
@@ -6,5 +6,6 @@
   <xacro:include filename="$(find linorobot2_description)/urdf/sensors/imu.urdf.xacro" />
   <xacro:include filename="$(find linorobot2_description)/urdf/sensors/generic_laser.urdf.xacro" />
-  <xacro:include filename="$(find linorobot2_description)/urdf/sensors/depth_sensor.urdf.xacro" />
+  <!--xacro:include filename="$(find linorobot2_description)/urdf/sensors/depth_sensor.urdf.xacro" /-->
+  <xacro:include filename="$(find linorobot2_description)/urdf/sensors/oakd_on_ptbase.urdf.xacro" />
   <xacro:include filename="$(find linorobot2_description)/urdf/controllers/skid_steer.urdf.xacro" />
   <xacro:base

File: linorobot2_description/urdf/sensors/imu.urdf.xacro (robot description, xacro)
@@ -5,5 +5,5 @@
       <parent link="base_link"/>
       <child link="imu_link"/>
-      <origin xyz="0 0 0" rpy="0 0 0"/>
+      <origin xyz="0 0.025 0.028" rpy="0 0 0"/>
     </joint>
     <gazebo reference="imu_link">

File: linorobot2_description/urdf/sensors/laser.urdf.xacro (robot description, xacro)
@@ -9,5 +9,5 @@
         </geometry>
         <material name="green">
-            <color rgba="0.003 0.639 0.223 1.0"/>
+            <color rgba="0.0 0.0 0.0 1.0"/>
         </material>
       </visual>
@@ -15,5 +15,5 @@
         <origin xyz="0 0 -0.025" rpy="0 0 0"/>
         <geometry>
-          <cylinder radius="0.0375" length="0.05"/>
+          <cylinder radius="0.0375" length="0.07"/>
         </geometry>
       </collision>
